Commit message: 6关节摔倒恢复

File: ddt_ros2_control/urdfs/tita_description/urdf/robot_4dot.urdf (robot description, URDF)
Before this commit: robot tita, 15 links, 14 joints
Joints:
- joint joint_left_leg_1: type revolute -> fixed
- joint joint_left_leg_4: type revolute -> fixed
- joint joint_right_leg_1: type revolute -> fixed
- joint joint_right_leg_4: type revolute -> fixed

File: ddt_ros2_control/urdfs/tita_description/urdf/robot_6dot.urdf (robot description, URDF)
Before this commit: robot tita, 15 links, 14 joints
Joints:
- joint joint_left_leg_1: type revolute -> fixed
- joint joint_right_leg_1: type revolute -> fixed
