Commit message: Add Andy robot locomotion configurations and environment setups
- Introduced new modules for the Andy robot, including environment configurations for flat, rough, and jump tasks.
- Implemented agent configurations for NP3O runners specific to Andy's locomotion tasks.
- Registered new Gym environments for Andy's locomotion tasks, including velocity and recovery scenarios.
- Developed flat and rough terrain configurations, incorporating domain randomization and reward shaping for effective training.
- Created jump environment configurations tailored for Andy's unique jumping capabilities.
- Established recovery configurations to enhance Andy's fall recovery strategies on both flat and rough terrains.
- Added support for terrain-aware locomotion, enabling a hybrid wheel-leg approach for stair climbing tasks.

File: ddt_ros2_control/urdfs/tita_description/urdf/robot_6dot.urdf (robot description, URDF)
Before this commit: robot tita, 15 links, 14 joints
Links:
- link base_link: geometry collision box size=0.47 0.3 0.19; visual mesh filename=/home/htw/ddt_lab/ddt_ros2_control/urdfs/andymini/meshes/ba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
