Commit message: add stairs

File: ddt_ros2_control/urdfs/tita6_description/urdf/robot.urdf (robot description, URDF)
Before this commit: robot tita, 15 links, 14 joints
Links:
- link base_link: geometry collision box size=0.47 0.3 0.19; visual mesh filename=../meshes/base_link.STL
- link imu_link: geometry collision box size=1.001 .001 .001; visual box size=0.001 0.001 0.001
- link left_leg_1: geometry visual mesh filename=../meshes/left_leg_1.STL
- link left_leg_2: geometry collision box size=0.26 0.09 0.05; visual mesh filename=../meshes/left_leg_2.STL
- link left_leg_3: geometry collision box size=0.2 0.07 0.05; visual mesh filename=../meshes/left_leg_3.STL
- link left_leg_4: geometry collision cylinder length=0.034 radius=0.0925; visual mesh filename=../meshes/left_leg_4.STL
- link right_leg_1: geometry visual mesh filename=../meshes/right_leg_1.STL
- link right_leg_2: geometry collision box size=0.26 0.09 0.05; visual mesh filename=../meshes/right_leg_2.STL
- link right_leg_3: geometry collision box size=0.2 0.07 0.05; visual mesh filename=../meshes/right_leg_3.STL
- link right_leg_4: geometry collision cylinder length=0.034 radius=0.0925; visual mesh filename=../meshes/right_leg_4.STL
Joints:
- joint joint_left_leg_1: type revolute -> fixed
- joint joint_right_leg_1: type revolute -> fixed

File: ddt_ros2_control/urdfs/tita6_description/xacro/robot.xacro (robot description, xacro)
@@ -4,5 +4,8 @@
 <!-- |    EDITING THIS FILE BY HAND IS NOT RECOMMENDED                                 | -->
 <!-- =================================================================================== -->
-<robot name="tita">
+<robot xmlns:xacro="http://wiki.ros.org/xacro" name="tita6">
+  <xacro:arg name="hw_env" default="none" />
+  <xacro:include filename="$(find tita6_description)/xacro/ros2control.xacro" />
+  <xacro:ros2control hw_env="$(arg hw_env)" />
   <material name="black">
     <color rgba="0.19607843137254902 0.19607843137254902 0.19607843137254902 1.0"/>
@@ -41,5 +44,5 @@
       <origin rpy="0 0 0" xyz="0 0 0"/>
       <geometry>
-        <mesh filename="package://tita_description/meshes/base_link.STL"/>
+        <mesh filename="package://tita6_description/meshes/base_link.STL"/>
       </geometry>
       <material name="black"/>
@@ -49,5 +52,5 @@
       <geometry>
         <box size="0.47 0.3 0.19"/>
-        <!-- <mesh filename="package://tita_description/collision/base_link1.stl" /> -->
+        <!-- <mesh filename="../collision/base_link1.stl" /> -->
       </geometry>
     </collision>
@@ -114,5 +117,5 @@
       <origin rpy="0 0 0" xyz="0 0 0"/>
       <geometry>
-        <box size=".001 .001 .001"/>
+        <box size="1.001 .001 .001"/>
       </geometry>
     </collision>
@@ -127,10 +130,10 @@
       <origin rpy="0 0 0" xyz="0 0 0"/>
       <geometry>
-        <mesh filename="package://tita_description/meshes/left_leg_1.STL"/>
-      </geometry>
-      <material name="black"/>
-    </visual>
-  </link>
-  <joint name="joint_left_leg_1" type="revolute">
+        <mesh filename="package://tita6_description/meshes/left_leg_1.STL"/>
+      </geometry>
+      <material name="black"/>
+    </visual>
+  </link>
+  <joint name="joint_left_leg_1" type="fixed">
     <origin rpy="1.5708 0 1.5708" xyz="0 0.0895 0"/>
     <parent link="base_link"/>
@@ -148,8 +151,14 @@
       <origin rpy="0 0 0" xyz="0 0 0"/>
       <geometry>
-        <mesh filename="package://tita_description/meshes/left_leg_2.STL"/>
-      </geometry>
-      <material name="black"/>
-    </visual>
+        <mesh filename="package://tita6_description/meshes/left_leg_2.STL"/>
+      </geometry>
+      <material name="black"/>
+    </visual>
+    <collision>
+      <origin rpy="0 0 0.2617993877991494" xyz="0.06 0.02 0"/>
+      <geometry>
+        <box size="0.26 0.09 0.05"/>
+      </geometry>
+    </collision>
   </link>
   <joint name="joint_left_leg_2" type="revolute">
@@ -164,10 +173,10 @@
       <origin rpy="0 0 0" xyz="0.095348 0.011698 0.001838"/>
       <mass value="0.57244"/>
-      <inertia ixx="0.000363" ixy="0.000237" ixz="-0.000109" iyy="0.004094 " iyz="0.000017" izz="0.004292"/>
-    </inertial>
-    <visual>
-      <origin rpy="0 0 0" xyz="0 0 0"/>
-      <geometry>
-        <mesh filename="package://tita_description/meshes/left_leg_3.STL"/>
+      <inertia ixx="0.000363" ixy="0.000237" ixz="-0.000109" iyy="0.004094" iyz="0.000017" izz="0.004292"/>
+    </inertial>
+    <visual>
+      <origin rpy="0 0 0" xyz="0 0 0"/>
+      <geometry>
+        <mesh filename="package://tita6_description/meshes/left_leg_3.STL"/>
       </geometry>
       <material name="black"/>
@@ -196,5 +205,5 @@
       <origin rpy="0 0 0" xyz="0 0 0"/>
       <geometry>
-        <mesh filename="package://tita_description/meshes/left_leg_4.STL"/>
+        <mesh filename="package://tita6_description/meshes/left_leg_4.STL"/>
       </geometry>
       <material name="black"/>
@@ -223,10 +232,10 @@
       <origin rpy="0 0 0" xyz="0 0 0"/>
       <geometry>
-        <mesh filename="package://tita_description/meshes/right_leg_1.STL"/>
-      </geometry>
-      <material name="black"/>
-    </visual>
-  </link>
-  <joint name="joint_right_leg_1" type="revolute">
+        <mesh filename="package://tita6_description/meshes/right_leg_1.STL"/>
+      </geometry>
+      <material name="black"/>
+    </visual>
+  </link>
+  <joint name="joint_right_leg_1" type="fixed">
     <origin rpy="1.5708 0 1.5708" xyz="0 -0.0895 0"/>
     <parent link="base_link"/>
@@ -244,8 +253,14 @@
       <origin rpy="0 0 0" xyz="0 0 0"/>
       <geometry>
-        <mesh filename="package://tita_description/meshes/right_leg_2.STL"/>
-      </geometry>
-      <material name="black"/>
-    </visual>
+        <mesh filename="package://tita6_description/meshes/right_leg_2.STL"/>
+      </geometry>
+      <material name="black"/>
+    </visual>
+    <collision>
+      <origin rpy="0 0 0.2617993877991494" xyz="0.06 0.02 0"/>
+      <geometry>
+        <box size="0.26 0.09 0.05"/>
+      </geometry>
+    </collision>
   </link>
   <joint name="joint_right_leg_2" type="revolute">
@@ -260,10 +275,10 @@
       <origin rpy="0 0 0" xyz="0.095348 0.011698 -0.001838"/>
       <mass value="0.57244"/>
-      <inertia ixx="0.000363" ixy="0.000237" ixz="0.000109" iyy="0.004094 " iyz="-0.000017" izz="0.004292"/>
-    </inertial>
-    <visual>
-      <origin rpy="0 0 0" xyz="0 0 0"/>
-      <geometry>
-        <mesh filename="package://tita_description/meshes/right_leg_3.STL"/>
+      <inertia ixx="0.000363" ixy="0.000237" ixz="0.000109" iyy="0.004094" iyz="-0.000017" izz="0.004292"/>
+    </inertial>
+    <visual>
+      <origin rpy="0 0 0" xyz="0 0 0"/>
+      <geometry>
+        <mesh filename="package://tita6_description/meshes/right_leg_3.STL"/>
       </geometry>
       <material name="black"/>
@@ -292,5 +307,5 @@
       <origin rpy="0 0 0" xyz="0 0 0"/>
       <geometry>
-        <mesh filename="package://tita_description/meshes/right_leg_4.STL"/>
+        <mesh filename="package://tita6_description/meshes/right_leg_4.STL"/>
       </geometry>
       <material name="black"/>
